File: PCB/ESP32-C3.kicad_sch (KiCad schematic)
At the start: 41 parts, among them J1 BattConn+, J2 BattConn-, SW1 TAK_6mm_THT, U1 USB-C-16P-SMD, U2 XT4052K421MR-G, U3 ESP32-C3, U4 RS3236-3.3YF5, X1 DPS_I2C, Y1 40MHz_S3240000151040

Commit message: gerber erstellt
Parts:
- X1: footprint Connector_PinHeader_2.54mm:PinHeader_1x04_P2.54mm_Vertical -> Connector_JST:JST_PH_B4B-PH-K_1x04_P2.00mm_Vertical
Changed lines of the file:
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@@
     (pin "1")
+  )
+  (symbol (lib_id "DPS_connectors:DPS_I2C") (at 149.86 168.91 0) (unit 1)
+    (in_bom yes) (on_board yes)
+    (property "Reference" "X1" (id 0) (at 148.59 163.83 0)
+      (effects (font (size 1.27 1.27)) (justify left))
+    )
+    (property "Value" "DPS_I2C" (id 1) (at 148.59 176.53 0)
+      (effects (font (size 1.27 1.27)) (justify left))
+    )
+    (property "Footprint" "Connector_JST:JST_PH_B4B-PH-K_1x04_P2.00mm_Vertical" (id 2) (at 148.59 163.83 0)
+      (effects (font (size 1.27 1.27)) hide)
+    )
+    (property "Datasheet" "https://datasheet.lcsc.com/lcsc/2009131335_CAX-PH-4A_C722775.pdf" (id 3) (at 149.225 162.56 0)
+      (effects (font (size 1.27 1.27)) hide)
+    )
+    (property "LCSC" "C722775" (id 4) (at 149.86 178.435 0)
+      (effects (font (size 1.27 1.27)) hide)
+    )
+    (pin "1")
+    (pin "2")
+    (pin "3")
+    (pin "4")
   )
   (symbol (lib_id "power:VCC") (at 119.38 29.21 0) (unit 1)
@@
     (pin "2")
   )
-  (symbol (lib_id "DPS_connectors:DPS_I2C") (at 149.86 168.91 0) (unit 1)
-    (in_bom yes) (on_board yes)
-    (property "Reference" "X1" (id 0) (at 148.59 163.83 0)
-      (effects (font (size 1.27 1.27)) (justify left))
-    )
-    (property "Value" "DPS_I2C" (id 1) (at 148.59 176.53 0)
-      (effects (font (size 1.27 1.27)) (justify left))
-    )
-    (property "Footprint" "Connector_PinHeader_2.54mm:PinHeader_1x04_P2.54mm_Vertical" (id 2) (at 148.59 163.83 0)
-      (effects (font (size 1.27 1.27)) hide)
-    )
-    (property "Datasheet" "https://datasheet.lcsc.com/lcsc/2009131335_CAX-PH-4A_C722775.pdf" (id 3) (at 149.225 162.56 0)
-      (effects (font (size 1.27 1.27)) hide)
-    )
-    (property "LCSC" "C722775" (id 4) (at 149.86 178.435 0)
-      (effects (font (size 1.27 1.27)) hide)
-    )
-    (pin "1")
-    (pin "2")
-    (pin "3")
-    (pin "4")
-  )
   (symbol (lib_id "power:GND") (at 119.38 59.69 0) (unit 1)
     (in_bom yes) (on_board yes) (fields_autoplaced)
@@
       (reference "U4") (unit 1) (value "RS3236-3.3YF5") (footprint "Package_TO_SOT_SMD:SOT-23-5")
     )
-    (path "/dec8301c-2558-4292-ad58-1d6c5e666965"
-      (reference "X1") (unit 1) (value "DPS_I2C") (footprint "Connector_PinHeader_2.54mm:PinHeader_1x04_P2.54mm_Vertical")
+    (path "/c70ab39b-441a-4f4b-97f0-87cbc795ab44"
+      (reference "X1") (unit 1) (value "DPS_I2C") (footprint "Connector_JST:JST_PH_B4B-PH-K_1x04_P2.00mm_Vertical")
     )
     (path "/8fa450c3-31b4-44e5-b47c-bc70761282fb"
