File: PCB/Version 1/_autosave-ESP32-C3.kicad_pcb (KiCad board)
At the start: 4 copper layers, 28.3 x 28.7 mm, 50 parts, among them J1 HCZZ0039-3, J2 DPS_PPS_Right_Angle, SW1 TS-1187A-B-A-B, SW2 TS-1187A-B-A-B, U1 USB-C-16P-SMD, U2 BQ24073RGTR, U3 ESP32-C3, U5 WL9003S5-33, Y1 40MHz_S3240000151040

Commit message: update
Other:
- copper layers 4 -> 2
Changed lines of the file:
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@@
 	(generator_version "8.0")
 	(general
-		(thickness 1.6062)
+		(thickness 1.6)
 		(legacy_teardrops no)
 	)
 	(paper "A4")
 	(layers
-		(0 "F.Cu" signal "Front.Cu")
-		(1 "In1.Cu" power "GND1.Cu")
-		(2 "In2.Cu" power "GND2.Cu")
-		(31 "B.Cu" signal "Back.Cu")
+		(0 "F.Cu" signal)
+		(31 "B.Cu" power)
 		(32 "B.Adhes" user "B.Adhesive")
 		(33 "F.Adhes" user "F.Adhesive")
@@
 			)
 			(layer "dielectric 1"
-				(type "prepreg")
-				(thickness 0.2104)
-				(material "FR4")
-				(epsilon_r 4.5)
-				(loss_tangent 0.02)
-			)
-			(layer "In1.Cu"
-				(type "copper")
-				(thickness 0.0152)
-			)
-			(layer "dielectric 2"
 				(type "core")
-				(thickness 1.065)
-				(material "FR4")
-				(epsilon_r 4.5)
-				(loss_tangent 0.02)
-			)
-			(layer "In2.Cu"
-				(type "copper")
-				(thickness 0.0152)
-			)
-			(layer "dielectric 3"
-				(type "prepreg")
-				(thickness 0.2104)
+				(thickness 1.51)
 				(material "FR4")
 				(epsilon_r 4.5)
@@
 		)
 	)
+	(dimension
+		(type aligned)
+		(layer "F.SilkS")
+		(pts
+			(xy 153.825137 96.3) (xy 153.836327 67.6)
+		)
+		(height 6.05706)
+		(gr_text "28,7 mm"
+			(at 158.737792 81.951914 89.97766064)
+			(layer "F.SilkS")
+			(effects
+				(font
+					(size 1 1)
+					(thickness 0.15)
+				)
+			)
+		)
+		(format
+			(prefix "")
+			(suffix "")
+			(units 2)
+			(units_format 1)
+			(precision 4) suppress_zeroes)
+		(style
+			(thickness 0.15)
+			(arrow_length 1.27)
+			(text_position_mode 0)
+			(extension_height 0.58642)
+			(extension_offset 0.5) keep_text_aligned)
+	)
+	(dimension
+		(type aligned)
+		(layer "F.SilkS")
+		(pts
+			(xy 128.974874 92.8) (xy 157.317737 92.825171)
+		)
+		(height 6.519419)
+		(gr_text "28,3 mm"
+			(at 143.141537 98.182002 359.9491142)
+			(layer "F.SilkS")
+			(effects
+				(font
+					(size 1 1)
+					(thickness 0.15)
+				)
+			)
+		)
+		(format
+			(prefix "")
+			(suffix "")
+			(units 2)
+			(units_format 1)
+			(precision 4)
+			(override_value "28,3") suppress_zeroes)
+		(style
+			(thickness 0.15)
+			(arrow_length 1.27)
+			(text_position_mode 0)
+			(extension_height 0.58642)
+			(extension_offset 0.5) keep_text_aligned)
+	)
 	(segment
