File: PCB/Version 2/ESP32-C3-V2.kicad_pcb (KiCad board)
At the start: 4 copper layers, 28.3 x 28.7 mm, 50 parts, among them J1 HCZZ0039-3, J2 DPS_PPS_Right_Angle, SW1 TS-1187A-B-A-B, SW2 TS-1187A-B-A-B, U1 USB-C-16P-SMD, U2 BQ24073RGTR, U3 ESP32-C3, U5 WL9003S5-33, Y1 40MHz_S3240000151040

Commit message: Working on Version 2
Parts:
- removed C14, C15, C19: 1u_0402_X5R_25V, Capacitor_SMD:C_0402_1005Metric
- removed C20, C21: 4u7_0402_X5R _10V, Capacitor_SMD:C_0402_1005Metric
- removed D4: 0603_WHITE, LED_SMD:LED_0603_1608Metric
- removed D5: 0603_RED, LED_SMD:LED_0603_1608Metric
- removed J1: HCZZ0039-3, Connector_JST:JST_SH_SM03B-SRSS-TB_1x03-1MP_P1.00mm_Horizontal
- removed L2: 2nH_0403_900mA, Resistor_SMD:R_0402_1005Metric
- removed SW1: TS-1187A-B-A-B, switch:SW_SPST_TL3305B
- added C10: 4u7_0402_X5R _10V, Capacitor_SMD:C_0402_1005Metric, F.Cu at (121.5, 72.0)
- added C8: 1u_0402_X5R_25V, Capacitor_SMD:C_0402_1005Metric, F.Cu at (121.5, 68.1)
- added D2: 0603_RED, LED_SMD:LED_0603_1608Metric, F.Cu at (121.6, 76.4)
- added D3: 0603_WHITE, LED_SMD:LED_0603_1608Metric, F.Cu at (121.6, 79.0)
- added J3: HCZZ0001-4, Connector_JST:JST_GH_SM04B-GHS-TB_1x04-1MP_P1.25mm_Horizontal, F.Cu at (101.4, 91.8)
- added Q1: WPM2031-3/TR, Package_TO_SOT_SMD:SOT-723, F.Cu at (132.5, 54.2)
- added R19: 10k_0402, Resistor_SMD:R_0402_1005Metric, F.Cu at (118.2, 91.0)
- added R20: 10k_0402, Resistor_SMD:R_0402_1005Metric, F.Cu at (118.6, 70.1)
- added R21: 3k_0402, Resistor_SMD:R_0402_1005Metric, F.Cu at (118.6, 72.1)
- added R22: 10k_0402, Resistor_SMD:R_0402_1005Metric, F.Cu at (118.6, 74.1)
- added U4: BQ24073RGTR, Package_DFN_QFN:VQFN-16-1EP_3x3mm_P0.5mm_EP1.6x1.6mm, F.Cu at (116.9, 77.8)
- C12: value 10n_0402_X7R_50V -> 100n_0402_X7R_16V
- C4: value 100n_0402_X7R_16V -> 1u_0402_X5R_25V
- C9: value 1u_0402_X5R_25V -> 4u7_0402_X5R _10V
- J2: value DPS_PPS_Right_Angle -> DPS_PPS; footprint Connector_JST:JST_PH_S2B-PH-K_1x02_P2.00mm_Horizontal -> Connector_JST:JST_PH_B2B-PH-K_1x02_P2.00mm_Vertical
- R1, R5, R6: value 5k1_0402 -> 10k_0402
- R10, R9: value 2k0_0402 -> 10k_0402
- R11: value 10k_0402 -> 1k5_0603; footprint Resistor_SMD:R_0402_1005Metric -> Resistor_SMD:R_0603_1608Metric
- R12: value 120_0402 -> 330_0402
- R13, R14: value 120_0402 -> 100k_0402
- R15: value 1k5_0603 -> 1M_0402; footprint Resistor_SMD:R_0603_1608Metric -> Resistor_SMD:R_0402_1005Metric
- R17: value 5k1_0402 -> 3k_0402
- R18: value 5k1_0402 -> 1k_0402
- R4: value 5k1_0402 -> 100_0402
- R7, R8: value 5k1_0402 -> 330_0402
- U2: value BQ24073RGTR -> DS8561-33S5; footprint Package_DFN_QFN:VQFN-16-1EP_3x3mm_P0.5mm_EP1.6x1.6mm -> Package_TO_SOT_SMD:SOT-23-5
- U5: value WL9003S5-33 -> SKCL3130ME
- moved R8 44.2 mm to (116.4, 54.1), turned to 0 degrees
- moved R7 43.8 mm to (116.4, 52.1), turned to 0 degrees
- moved R12 39.5 mm to (116.4, 56.1)
- moved C12 39.3 mm to (132.7, 56.2)
- moved U5 38.0 mm to (107.8, 65.4)
- moved C4 37.0 mm to (121.5, 66.1), turned to 0 degrees
- moved U2 33.6 mm to (108.9, 77.2)
- moved C1 32.3 mm to (118.2, 93.0), turned to 0 degrees
- moved R14 31.0 mm to (129.8, 55.4), turned to 0 degrees
- moved R13 30.2 mm to (129.8, 53.4), turned to 0 degrees
- moved R1 30.2 mm to (118.2, 87.0), turned to 0 degrees
- moved R6 29.3 mm to (118.2, 89.0), turned to 0 degrees
- moved J2 28.7 mm to (107.0, 70.1), turned to 0 degrees
- moved R16 26.6 mm to (115.7, 74.1), turned to 0 degrees
- moved R9 26.2 mm to (115.7, 70.1), turned to 0 degrees
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Connections:
- C1 pad 1: GND -> +3.3V
- C1 pad 2: EXTI -> GND
- C12 pad 1: +3.3V -> EN_ADC
- C12 pad 2: GND -> Net-(Q1-G)
- C4 pad 1: GND -> Net-(U5-Vin)
- C4 pad 2: +3.3V -> Earth
- C7 pad 2: Net-(C7-Pad2) -> +3.3V
- C9 pad 1: +3.3V -> +BATT
- J2 pad 1: +BATT -> Earth
- J2 pad 2: GND -> +BATT
- R1 pad 1: EXTI -> +3.3V
- R1 pad 2: +3.3V -> EXTI
- R10 pad 1: Net-(D4-A) -> VCC
- R10 pad 2: +3.3V -> EN2
- R11 pad 1: Net-(U2-TS) -> Net-(U4-ILIM)
- R13 pad 1: Grün -> Net-(Q1-D)
- R13 pad 2: Net-(D1-GK) -> ADC
- R14 pad 1: Blau -> ADC
- R14 pad 2: Net-(D1-BK) -> GND
- R15 pad 1: Net-(U2-ILIM) -> +BATT
- R15 pad 2: GND -> Net-(Q1-G)
- R16 pad 1: GND -> Net-(U4-ISET)
- R16 pad 2: EN1 -> GND
- R17 pad 1: EN2 -> Net-(D3-A)
- R17 pad 2: +3.3V -> VCC
- R18 pad 1: Net-(U2-ISET) -> Net-(U2-Vin)
- R18 pad 2: GND -> Net-(U2-EN)
- R4 pad 1: GND -> +BATT
- R4 pad 2: NCE -> Net-(U5-Vin)
- R5 pad 1: GND -> VCC
- R5 pad 2: TMR -> NCE
- R6 pad 1: CHIP_EN -> +3.3V
- R6 pad 2: +3.3V -> GPIO8
- R7 pad 1: MCU_SCL -> Blau
- R7 pad 2: +3.3V -> Net-(D1-BK)
- R8 pad 1: MCU_SDA -> Grün
- R8 pad 2: +3.3V -> Net-(D1-GK)
- R9 pad 1: Net-(D5-A) -> EN1
- R9 pad 2: +3.3V -> GND
- U2 pad 1: Net-(U2-TS) -> Net-(U2-Vin)
- U2 pad 2: +BATT -> GND
- U2 pad 3: +BATT -> Net-(U2-EN)
- U2 pad 4: NCE -> unconnected-(U2-NC-Pad4)
- U2 pad 5: EN2 -> +3.3V
- U3 pad 12: unconnected-(U3-MTCK-Pad12) -> EN_ADC
- U3 pad 14: TD -> GPIO8
- U3 pad 16: TMR -> VCC_Sensor
- U3 pad 19: NPGOOD -> unconnected-(U3-SPIHD-Pad19)
- U3 pad 2: Net-(C7-Pad2) -> +3.3V
- U3 pad 20: NCHG -> ADC
- U3 pad 3: Net-(C7-Pad2) -> +3.3V
- U5 pad 1: Net-(U5-EN) -> unconnected-(U5-VT-Pad1)
- U5 pad 2: GND -> Earth
- U5 pad 3: Net-(U5-EN) -> Net-(U5-Vin)
- U5 pad 4: unconnected-(U5-NC-Pad4) -> GND
- U5 pad 5: +3.3V -> GND
Routing:
- net +3.3V: track 111.5 -> 0.00 mm, vias 10 -> 0
- net GND: track 45.5 -> 0.00 mm, vias 46 -> 0
- net NCHG: track 40.4 -> 0.00 mm, vias 2 -> 0
- net VCC: track 35.6 -> 0.00 mm
- net MCU_SDA: track 32.8 -> 0.00 mm, vias 2 -> 0
- net NPGOOD: track 32.6 -> 0.00 mm, vias 2 -> 0
- net MCU_SCL: track 31.7 -> 0.00 mm, vias 2 -> 0
- net TMR: track 30.3 -> 0.00 mm, vias 2 -> 0
- net Net-(U3-GPIO9): track 29.0 -> 0.00 mm, vias 4 -> 0
- net EXTI: track 25.4 -> 0.00 mm
- net Grün: track 23.3 -> 0.00 mm, vias 2 -> 0
- net EN1: track 19.9 -> 0.00 mm, vias 2 -> 0
- net EN2: track 18.1 -> 0.00 mm, vias 2 -> 0
- net USB_D+: track 17.6 -> 0.00 mm
- net TD: track 17.6 -> 0.00 mm, vias 2 -> 0
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- added copper zone on In2.Cu, net +3.3V
- added copper zone on In1.Cu, net GND
- removed copper zone on F.Cu, net +3.3V
- removed copper zone on F.Cu, net GND
Other:
- board text removed: "+"
- board text removed: "-"
- board text removed: "A.S. V1 W-Charger 06.2024"
- board text removed: "B"
- board text removed: "Charging"
- board text removed: "D"
- board text removed: "GND SCL SDA"
- board text removed: "Pow."
- board text removed: "Power"

Commit message: Version 2
Parts:
- removed R10, R22, R9: 10k_0402, Resistor_SMD:R_0402_1005Metric
- added C13: 100n_0402_X7R_16V, Capacitor_SMD:C_0402_1005Metric, F.Cu at (139.1, 86.8)
- R5: value 10k_0402 -> 1k_0402
- moved J3 52.3 mm to (150.9, 74.9), turned to 180 degrees
- moved R7 44.5 mm to (139.6, 90.1), turned to 180 degrees
- moved R8 43.7 mm to (139.6, 91.1), turned to 180 degrees
- moved R12 40.3 mm to (139.6, 89.1), turned to 180 degrees
- moved U5 39.0 mm to (143.2, 81.8), turned to -90 degrees
- moved J2 36.9 mm to (143.6, 75.0), turned to 180 degrees
- moved D3 31.3 mm to (92.1, 68.4)
- moved R13 30.3 mm to (130.7, 83.6), turned to 90 degrees
- moved R1 30.2 mm to (148.4, 86.9), turned to -90 degrees
- moved R4 29.5 mm to (142.1, 79.2)
- moved R19 29.4 mm to (147.4, 86.9), turned to -90 degrees
- moved Q1 29.4 mm to (132.2, 83.6), turned to -90 degrees
- moved R5 29.2 mm to (138.1, 86.8), turned to -90 degrees
- moved C1 28.6 mm to (146.8, 92.8)
- moved R14 28.3 mm to (129.7, 83.6), turned to -90 degrees
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Connections:
- C10 pad 1: Net-(U2-Vin) -> OUT
- R13 pad 2: ADC -> Net-(R13-Pad2)
- R14 pad 1: ADC -> Net-(R13-Pad2)
- R17 pad 2: VCC -> OUT
- R18 pad 1: Net-(U2-Vin) -> OUT
- R21 pad 2: VCC -> OUT
- R5 pad 1: VCC -> Net-(R13-Pad2)
- R5 pad 2: NCE -> ADC
- U2 pad 1: Net-(U2-Vin) -> OUT
- U3 pad 16: VCC_Sensor -> EN2
- U3 pad 18: Rot -> ADC
- U3 pad 19: unconnected-(U3-SPIHD-Pad19) -> EN1
- U3 pad 20: ADC -> TD
- U3 pad 21: EN2 -> unconnected-(U3-SPICS0-Pad21)
- U3 pad 22: EN1 -> Rot
- U3 pad 8: unconnected-(U3-GPIO3-Pad8) -> VCC_Sensor
- U4 pad 10: Net-(U2-Vin) -> OUT
- U4 pad 11: Net-(U2-Vin) -> OUT
- U4 pad 15: Net-(U4-TD) -> TD
Other:
- board size 28.3 x 28.7 mm -> 28.1 x 24.5 mm

Commit message: V2 für Kontrolle fertig
Parts:
- added C14: 1u_0402_X5R_25V, Capacitor_SMD:C_0402_1005Metric, F.Cu at (150.1, 86.9)
- moved D3 46.1 mm to (137.8, 74.3), turned to 90 degrees
- moved R17 44.6 mm to (136.5, 73.8), turned to -90 degrees
- moved R21 37.3 mm to (132.4, 73.9), turned to -90 degrees
- moved D2 35.8 mm to (131.0, 74.4), turned to 90 degrees
- moved R14 4.74 mm to (134.2, 85.1), turned to 0 degrees
- moved R15 2.28 mm to (130.8, 83.6), turned to -90 degrees
- moved R13 2.12 mm to (132.2, 85.1), turned to 0 degrees
- moved R3 1.40 mm to (136.5, 95.0)
- moved R5 0.86 mm to (137.6, 86.1), turned to 0 degrees
- moved J2 0.78 mm to (143.0, 75.5)
- moved J3 0.78 mm to (150.1, 75.0)
- moved C17 0.75 mm to (141.8, 94.2)
- moved Y1 0.72 mm to (144.4, 94.0)
- moved C16 0.71 mm to (147.0, 94.3)
- moved R1 0.70 mm to (149.1, 86.9)
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Routing:
- net GND: track 0.00 -> 27.6 mm, vias 0 -> 60
- net VCC: track 0.00 -> 24.4 mm
- net MCU_SDA: track 0.00 -> 17.1 mm
- net EN1: track 0.00 -> 16.1 mm, vias 0 -> 2
- net OUT: track 0.00 -> 13.8 mm, vias 0 -> 2
- net VCC_Sensor: track 0.00 -> 13.5 mm
- net +3.3V: track 0.00 -> 13.5 mm, vias 0 -> 16
- net Net-(U3-GPIO9): track 0.00 -> 12.9 mm, vias 0 -> 2
- net EN2: track 0.00 -> 12.8 mm, vias 0 -> 2
- net MCU_SCL: track 0.00 -> 12.7 mm
- net NCE: track 0.00 -> 12.3 mm, vias 0 -> 2
- net EN_ADC: track 0.00 -> 12.1 mm, vias 0 -> 2
- net +BATT: track 0.00 -> 11.8 mm, vias 0 -> 2
- net USB_D+: track 0.00 -> 10.9 mm
- net TD: track 0.00 -> 10.3 mm
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- added copper zone on F.Cu, net +3.3V
- added copper zone on F.Cu, net +BATT
- added copper zone on F.Cu, net Earth
- added copper zone on F.Cu, net GND
- added copper zone on F.Cu, net OUT
Other:
- board size 28.1 x 24.5 mm -> 28.1 x 24.4 mm
- board text added: "+"
- board text added: "-"
- board text added: "A.S. V2 W-Charger 07.24"
- board text added: "Charg"
- board text added: "GND"
- board text added: "Power"
- board text added: "SCL"
- board text added: "SDA"
- board text added: "VCC"
